File: electrical/Stepper-Motor-Driver/tests/H-Bridge Arduino Testing Circuit/circuit/Testing Circuit.kicad_sch (KiCad schematic)
At the start: 70 parts, among them M1 Stepper_Motor_bipolar, Q1 IRF530NPBF, Q2 IRF530NPBF, Q3 IRF530NPBF, Q4 IRF530NPBF, Q5 IRF530NPBF, Q6 IRF530NPBF, Q7 IRF530NPBF, Q8 IRF530NPBF, U1 UCC27710D, U2 UCC27710D, U3 UCC27710D, U4 UCC27710D

Commit message: Adding capacitors to reduce ringing from parasitic wire inductance
Parts:
- added C11, C12: 150nF, symbol Device:C
Connections:
- net at C1.2, M1.2 (-), Q1.3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: now also C11.1
- net at C3.2, M1.3, Q5.3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: now also C12.1
- net at C9.2, R2.1, U2.3 (LI): no longer A1.D23
- net at R2.2: now also A1.D23
- net at C4.1, M1.4, Q7.3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: now also C12.2
- net at C2.1, M1.1, Q3.2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: now also C11.2
- net at C10.2, R1.1, U2.2 (HI): no longer A1.D22
- net at R1.2: now also A1.D22
Changed lines of the file:
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@@
 	)
 	(junction
-		(at 69.85 120.65)
+		(at 149.86 87.63)
 		(diameter 0)
 		(color 0 0 0 0)
@@
 	)
 	(junction
+		(at 157.48 86.36)
+		(diameter 0)
+		(color 0 0 0 0)
+	)
+	(junction
+		(at 162.56 90.17)
+		(diameter 0)
+		(color 0 0 0 0)
+	)
+	(junction
 		(at 220.98 44.45)
 		(diameter 0)
@@
 	)
 	(junction
-		(at 220.98 34.29)
+		(at 163.83 97.79)
 		(diameter 0)
 		(color 0 0 0 0)
 	)
 	(junction
-		(at 217.17 39.37)
+		(at 220.98 34.29)
 		(diameter 0)
 		(color 0 0 0 0)
 	)
 	(junction
-		(at 31.75 83.82)
+		(at 217.17 39.37)
 		(diameter 0)
 		(color 0 0 0 0)
 	)
 	(junction
-		(at 67.31 120.65)
+		(at 31.75 83.82)
 		(diameter 0)
 		(color 0 0 0 0)
@@
 	(wire
 		(pts
-			(xy 162.56 97.79) (xy 165.1 97.79)
+			(xy 162.56 97.79) (xy 163.83 97.79)
 		)
 		(stroke
@@
 	(wire
 		(pts
+			(xy 67.31 128.27) (xy 67.31 132.08)
+		)
+		(stroke
+			(width 0)
+			(type default)
+		)
+	)
+	(wire
+		(pts
 			(xy 165.1 97.79) (xy 165.1 87.63)
 		)
@@
 	(wire
 		(pts
+			(xy 157.48 86.36) (xy 157.48 85.09)
+		)
+		(stroke
+			(width 0)
+			(type default)
+		)
+	)
+	(wire
+		(pts
 			(xy 67.31 76.2) (xy 67.31 83.82)
 		)
@@
 	(wire
 		(pts
-			(xy 162.56 92.71) (xy 162.56 85.09)
+			(xy 162.56 92.71) (xy 162.56 90.17)
 		)
 		(stroke
@@
 	(wire
 		(pts
-			(xy 67.31 120.65) (xy 67.31 132.08)
-		)
-		(stroke
-			(width 0)
-			(type default)
-		)
-	)
-	(wire
-		(pts
 			(xy 157.48 85.09) (xy 121.92 85.09)
 		)
@@
 	(wire
 		(pts
+			(xy 162.56 90.17) (xy 163.83 90.17)
+		)
+		(stroke
+			(width 0)
+			(type default)
+		)
+	)
+	(wire
+		(pts
 			(xy 266.7 26.67) (xy 266.7 34.29)
 		)
@@
 	(wire
 		(pts
-			(xy 69.85 120.65) (xy 69.85 132.08)
-		)
-		(stroke
-			(width 0)
-			(type default)
-		)
-	)
-	(wire
-		(pts
 			(xy 71.12 67.31) (xy 78.74 67.31)
 		)
@@
 	(wire
 		(pts
+			(xy 149.86 87.63) (xy 119.38 87.63)
+		)
+		(stroke
+			(width 0)
+			(type default)
+		)
+	)
+	(wire
+		(pts
 			(xy 15.24 93.98) (xy 15.24 92.71)
 		)
@@
 	(wire
 		(pts
+			(xy 69.85 128.27) (xy 69.85 132.08)
+		)
+		(stroke
+			(width 0)
+			(type default)
+		)
+	)
+	(wire
+		(pts
 			(xy 207.01 50.8) (xy 207.01 58.42)
 		)
@@
 	(wire
 		(pts
-			(xy 152.4 87.63) (xy 119.38 87.63)
+			(xy 152.4 87.63) (xy 149.86 87.63)
 		)
 		(stroke
@@
 	(wire
 		(pts
+			(xy 149.86 86.36) (xy 149.86 87.63)
+		)
+		(stroke
+			(width 0)
+			(type default)
+		)
+	)
+	(wire
+		(pts
+			(xy 163.83 97.79) (xy 165.1 97.79)
+		)
+		(stroke
+			(width 0)
+			(type default)
+		)
+	)
+	(wire
+		(pts
 			(xy 97.79 53.34) (xy 97.79 58.42)
 		)
@@
 	(wire
 		(pts
-			(xy 157.48 87.63) (xy 157.48 85.09)
+			(xy 157.48 87.63) (xy 157.48 86.36)
 		)
 		(stroke
@@
 	(wire
 		(pts
+			(xy 162.56 90.17) (xy 162.56 85.09)
+		)
+		(stroke
+			(width 0)
+			(type default)
+		)
+	)
+	(wire
+		(pts
 			(xy 280.67 21.59) (xy 280.67 88.9)
 		)
@@
 	)
 	(symbol
+		(lib_id "Device:C")
+		(at 153.67 86.36 90)
+		(unit 1)
+		(body_style 1)
+		(exclude_from_sim no)
+		(in_bom yes)
+		(on_board yes)
+		(in_pos_files yes)
+		(dnp no)
+		(fields_autoplaced yes)
+		(property "Reference" "C11"
+			(at 153.67 78.74 90)
+			(show_name no)
+			(do_not_autoplace no)
+			(effects
+				(font
+					(size 1.27 1.27)
+				)
+			)
+		)
+		(property "Value" "150nF"
+			(at 153.67 81.28 90)
+			(show_name no)
+			(do_not_autoplace no)
+			(effects
+				(font
+					(size 1.27 1.27)
+				)
+			)
+		)
+		(property "Footprint" ""
+			(at 157.48 85.3948 0)
+			(hide yes)
+			(show_name no)
+			(do_not_autoplace no)
+			(effects
+				(font
+					(size 1.27 1.27)
+				)
+			)
+		)
+		(property "Datasheet" ""
+			(at 153.67 86.36 0)
+			(hide yes)
+			(show_name no)
+			(do_not_autoplace no)
+			(effects
+				(font
+					(size 1.27 1.27)
+				)
+			)
+		)
+		(property "Description" "Unpolarized capacitor"
+			(at 153.67 86.36 0)
+			(hide yes)
+			(show_name no)
+			(do_not_autoplace no)
+			(effects
+				(font
+					(size 1.27 1.27)
+				)
+			)
+		)
+		(pin "1"
+		)
+		(pin "2"
+		)
+		(instances
+			(project "Testing Circuit"
+				(path "/c25060f1-f2f3-4cbd-b6ee-5f66e19502f5"
+					(reference "C11")
+					(unit 1)
+				)
+			)
+		)
+	)
+	(symbol
 		(lib_id "Device:R")
 		(at 227.33 88.9 0)
@@
 					(unit 1)
 				)
+			)
+		)
+	)
+	(symbol
+		(lib_id "Device:C")
+		(at 163.83 93.98 0)
+		(unit 1)
+		(body_style 1)
+		(exclude_from_sim no)
+		(in_bom yes)
+		(on_board yes)
+		(in_pos_files yes)
+		(dnp no)
+		(fields_autoplaced yes)
+		(property "Reference" "C12"
+			(at 167.64 92.7099 0)
+			(show_name no)
+			(do_not_autoplace no)
+			(effects
+				(font
+					(size 1.27 1.27)
+				)
+				(justify left)
+			)
+		)
+		(property "Value" "150nF"
+			(at 167.64 95.2499 0)
+			(show_name no)
+			(do_not_autoplace no)
+			(effects
+				(font
+					(size 1.27 1.27)
+				)
+				(justify left)
+			)
+		)
+		(property "Footprint" ""
+			(at 164.7952 97.79 0)
+			(hide yes)
+			(show_name no)
+			(do_not_autoplace no)
+			(effects
+				(font
+					(size 1.27 1.27)
+				)
+			)
+		)
+		(property "Datasheet" ""
+			(at 163.83 93.98 0)
+			(hide yes)
+			(show_name no)
+			(do_not_autoplace no)
+			(effects
+				(font
+					(size 1.27 1.27)
+				)
+			)
+		)
+		(property "Description" "Unpolarized capacitor"
+			(at 163.83 93.98 0)
+			(hide yes)
+			(show_name no)
+			(do_not_autoplace no)
+			(effects
+				(font
+					(size 1.27 1.27)
+				)
+			)
+		)
+		(pin "1"
+		)
+		(pin "2"
+		)
+		(instances
+			(project "Testing Circuit"
+				(path "/c25060f1-f2f3-4cbd-b6ee-5f66e19502f5"
+					(reference "C12")
+					(unit 1)
+				)
