File: electrical/Stepper-Motor-Driver/circuits/Stepper Motor Driver.kicad_sch (KiCad schematic)
At the start: 17 parts, among them M2 Stepper_Motor_bipolar

Commit message: Current sensing circuit
Parts:
- removed M2: Stepper_Motor_bipolar, symbol Motor:Stepper_Motor_bipolar
- added J1: Screw_Terminal_01x04, symbol Connector:Screw_Terminal_01x04
Connections:
- net H-Bridge Controller A/HIA renamed H-Bridge Controller A/HI1
- net H-Bridge Controller A/HIB renamed H-Bridge Controller A/HI2
- net H-Bridge Controller A/LIA renamed H-Bridge Controller A/LI1
- net H-Bridge Controller A/LIB renamed H-Bridge Controller A/LI2
- net H-Bridge Controller B/HIA renamed H-Bridge Controller B/HI1
- net H-Bridge Controller B/HIB renamed H-Bridge Controller B/HI2
- net H-Bridge Controller B/LIA renamed H-Bridge Controller B/LI1
- net H-Bridge Controller B/LIB renamed H-Bridge Controller B/LI2
- net HIA1 renamed HI1A
- net HIA2 renamed LI2B
- net HIB1 renamed HI2A
- net HIB2 renamed LI1B
- net LIA1 renamed LI1A
- net LIA2 renamed HI2B
- net LIB1 renamed LI2A
- net LIB2 renamed HI1B
- new net Current Sensor A/IN-: J1.1 (Pin_1)
- new net Current Sensor B/IN-: J1.3 (Pin_3)
- new net H-Bridge Controller A/BR2: J1.2 (Pin_2)
- new net H-Bridge Controller B/BR2: J1.4 (Pin_4)
Other:
- sheet H-Bridge Controller 1 renamed H-Bridge Controller A
- sheet H-Bridge Controller 2 renamed H-Bridge Controller B
- added sheet Current Sensor A (Current Sensor.kicad_sch)
- added sheet Current Sensor B (Current Sensor.kicad_sch)
- sheet H-Bridge Controller A ports: added BR1, BR2, HI1, HI2, LI1, LI2; removed BRA, BRB, HIA, HIB, LIA, LIB
- sheet H-Bridge Controller B ports: added BR1, BR2, HI1, HI2, LI1, LI2; removed BRA, BRB, HIA, HIB, LIA, LIB
- note added: "Connect terminal 1 to coil A and back to terminal 2. Connect terminal 3 to coil B and back to terminal 4."
- note added: "H-Bridge for coil A"
- note added: "H-Bridge for coil B"
- moved on the sheet: C19, C20, C21, C22, R5, R6, R7, R8

Commit message: Through holes for FPGA
Parts:
- added J1, J2: Conn_01x22_Socket, Connector_PinSocket_2.54mm:PinSocket_1x22_P2.54mm_Vertical, symbol Connector:Conn_01x22_Socket
Changed lines of the file:
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@@
+	)
+	(symbol
+		(lib_id "Connector:Conn_01x22_Socket")
+		(at 55.88 165.1 90)
+		(unit 1)
+		(body_style 1)
+		(exclude_from_sim no)
+		(in_bom yes)
+		(on_board yes)
+		(in_pos_files yes)
+		(dnp no)
+		(property "Reference" "J2"
+			(at 57.15 162.56 90)
+			(show_name no)
+			(do_not_autoplace no)
+			(effects
+				(font
+					(size 1.27 1.27)
+				)
+			)
+		)
+		(property "Value" "Conn_01x22_Socket"
+			(at 57.15 160.02 90)
+			(show_name no)
+			(do_not_autoplace no)
+			(effects
+				(font
+					(size 1.27 1.27)
+				)
+			)
+		)
+		(property "Footprint" "Connector_PinSocket_2.54mm:PinSocket_1x22_P2.54mm_Vertical"
+			(at 55.88 164.084 90)
+			(show_name no)
+			(do_not_autoplace no)
+			(effects
+				(font
+					(size 1.27 1.27)
+				)
+			)
+		)
+		(property "Datasheet" ""
+			(at 55.88 165.1 0)
+			(hide yes)
+			(show_name no)
+			(do_not_autoplace no)
+			(effects
+				(font
+					(size 1.27 1.27)
+				)
+			)
+		)
+		(property "Description" "Generic connector, single row, 01x22, script generated"
+			(at 55.88 165.1 0)
+			(hide yes)
+			(show_name no)
+			(do_not_autoplace no)
+			(effects
+				(font
+					(size 1.27 1.27)
+				)
+			)
+		)
+		(pin "16"
+		)
+		(pin "18"
+		)
+		(pin "1"
+		)
+		(pin "2"
+		)
+		(pin "10"
+		)
+		(pin "4"
+		)
+		(pin "11"
+		)
+		(pin "9"
+		)
+		(pin "3"
+		)
+		(pin "13"
+		)
+		(pin "15"
+		)
+		(pin "12"
+		)
+		(pin "6"
+		)
+		(pin "14"
+		)
+		(pin "7"
+		)
+		(pin "5"
+		)
+		(pin "8"
+		)
+		(pin "17"
+		)
+		(pin "20"
+		)
+		(pin "19"
+		)
+		(pin "22"
+		)
+		(pin "21"
+		)
+		(instances
+			(project "Stepper Motor Driver"
+				(path "/c25060f1-f2f3-4cbd-b6ee-5f66e19502f5"
+					(reference "J2")
+					(unit 1)
+				)
+			)
+		)
 	)
 	(symbol
@@
 					(unit 1)
 				)
+			)
+		)
+	)
+	(symbol
+		(lib_id "Connector:Conn_01x22_Socket")
+		(at 58.42 144.78 270)
+		(unit 1)
+		(body_style 1)
+		(exclude_from_sim no)
+		(in_bom yes)
+		(on_board yes)
+		(in_pos_files yes)
+		(dnp no)
+		(property "Reference" "J1"
+			(at 57.15 147.32 90)
+			(show_name no)
+			(do_not_autoplace no)
+			(effects
+				(font
+					(size 1.27 1.27)
+				)
+			)
+		)
+		(property "Value" "Conn_01x22_Socket"
+			(at 57.15 149.86 90)
+			(show_name no)
+			(do_not_autoplace no)
+			(effects
+				(font
+					(size 1.27 1.27)
+				)
+			)
+		)
+		(property "Footprint" "Connector_PinSocket_2.54mm:PinSocket_1x22_P2.54mm_Vertical"
+			(at 58.42 145.796 90)
+			(show_name no)
+			(do_not_autoplace no)
+			(effects
+				(font
+					(size 1.27 1.27)
+				)
+			)
+		)
+		(property "Datasheet" ""
+			(at 58.42 144.78 0)
+			(hide yes)
+			(show_name no)
+			(do_not_autoplace no)
+			(effects
+				(font
+					(size 1.27 1.27)
+				)
+			)
+		)
+		(property "Description" "Generic connector, single row, 01x22, script generated"
+			(at 58.42 144.78 0)
+			(hide yes)
+			(show_name no)
+			(do_not_autoplace no)
+			(effects
+				(font
+					(size 1.27 1.27)
+				)
+			)
+		)
+		(pin "16"
+		)
+		(pin "18"
+		)
+		(pin "1"
+		)
+		(pin "2"
+		)
+		(pin "10"
+		)
+		(pin "4"
+		)
+		(pin "11"
+		)
+		(pin "9"
+		)
+		(pin "3"
+		)
+		(pin "13"
+		)
+		(pin "15"
+		)
+		(pin "12"
+		)
+		(pin "6"
+		)
+		(pin "14"
+		)
+		(pin "7"
+		)
+		(pin "5"
+		)
+		(pin "8"
+		)
+		(pin "17"
+		)
+		(pin "20"
+		)
+		(pin "19"
+		)
+		(pin "22"
+		)
+		(pin "21"
+		)
+		(instances
+			(project "Stepper Motor Driver"
+				(path "/c25060f1-f2f3-4cbd-b6ee-5f66e19502f5"
+					(reference "J1")
+					(unit 1)
+				)

Commit message: Symbol cleanup and initial power section design
Parts:
- removed J1: Screw_Terminal_01x04, symbol Connector:Screw_Terminal_01x04
- added J3: Screw_Terminal_01x04, symbol Connector:Screw_Terminal_01x04
- C15, C16, C17, C18, C19, C20, C21, C22: footprint (none) -> Capacitor_SMD:C_1206_3216Metric
- R1, R2, R3, R4, R5, R6, R7, R8: footprint (none) -> Resistor_SMD:R_1206_3216Metric
Connections:
- net Current Sensor A/IN-: now also J3.1 (Pin_1)
- net Current Sensor B/IN-: now also J3.3 (Pin_3)
- net H-Bridge Controller A/BR2: now also J3.2 (Pin_2)
- net H-Bridge Controller B/BR2: now also J3.4 (Pin_4)
Other:
- added sheet Power (Power.kicad_sch)
Changed lines of the file:
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@@
-	)
-	(symbol
-		(lib_id "Connector:Screw_Terminal_01x04")
-		(at 140.97 76.2 90)
-		(unit 1)
-		(body_style 1)
-		(exclude_from_sim no)
-		(in_bom yes)
-		(on_board yes)
-		(in_pos_files yes)
-		(dnp no)
-		(fields_autoplaced yes)
-		(property "Reference" "J1"
-			(at 142.24 69.85 90)
-			(show_name no)
-			(do_not_autoplace no)
-			(effects
-				(font
-					(size 1.27 1.27)
-				)
-			)
-		)
-		(property "Value" "Screw_Terminal_01x04"
-			(at 142.24 72.39 90)
-			(show_name no)
-			(do_not_autoplace no)
-			(effects
-				(font
-					(size 1.27 1.27)
-				)
-			)
-		)
-		(property "Footprint" ""
-			(at 140.97 76.2 0)
-			(hide yes)
-			(show_name no)
-			(do_not_autoplace no)
-			(effects
-				(font
-					(size 1.27 1.27)
-				)
-			)
-		)
-		(property "Datasheet" ""
-			(at 140.97 76.2 0)
-			(hide yes)
-			(show_name no)
-			(do_not_autoplace no)
-			(effects
-				(font
-					(size 1.27 1.27)
-				)
-			)
-		)
-		(property "Description" "Generic screw terminal, single row, 01x04, script generated (kicad-library-utils/schlib/autogen/connector/)"
-			(at 140.97 76.2 0)
-			(hide yes)
-			(show_name no)
-			(do_not_autoplace no)
-			(effects
-				(font
-					(size 1.27 1.27)
-				)
-			)
-		)
-		(pin "1"
-		)
-		(pin "3"
-		)
-		(pin "4"
-		)
-		(pin "2"
-		)
-		(instances
-			(project "Stepper Motor Driver"
-				(path "/c25060f1-f2f3-4cbd-b6ee-5f66e19502f5"
-					(reference "J1")
-					(unit 1)
-				)
-			)
-		)
 	)
 	(symbol
@@
 			)
 		)
-		(property "Footprint" ""
+		(property "Footprint" "Capacitor_SMD:C_1206_3216Metric"
 			(at 259.08 53.6448 0)
 			(hide yes)
@@
 			)
 		)
-		(property "Footprint" ""
+		(property "Footprint" "Resistor_SMD:R_1206_3216Metric"
 			(at 50.292 59.69 90)
 			(hide yes)
@@
 			)
 		)
-		(property "Footprint" ""
+		(property "Footprint" "Resistor_SMD:R_1206_3216Metric"
 			(at 258.572 59.69 90)
 			(hide yes)
@@
 			)
 		)
-		(property "Footprint" ""
+		(property "Footprint" "Capacitor_SMD:C_1206_3216Metric"
 			(at 91.44 53.6448 0)
 			(hide yes)
@@
 			)
 		)
-		(property "Footprint" ""
+		(property "Footprint" "Capacitor_SMD:C_1206_3216Metric"
 			(at 50.8 53.6448 0)
 			(hide yes)
@@
 			)
 		)
-		(property "Footprint" ""
+		(property "Footprint" "Capacitor_SMD:C_1206_3216Metric"
 			(at 238.76 53.6448 0)
 			(hide yes)
@@
 			)
 		)
-		(property "Footprint" ""
+		(property "Footprint" "Capacitor_SMD:C_1206_3216Metric"
 			(at 199.39 53.6448 0)
 			(hide yes)
@@
 			)
 		)
-		(property "Footprint" ""
+		(property "Footprint" "Resistor_SMD:R_1206_3216Metric"
 			(at 29.972 59.69 90)
 			(hide yes)
@@
 			)
 		)
-		(property "Footprint" ""
+		(property "Footprint" "Resistor_SMD:R_1206_3216Metric"
 			(at 217.932 59.69 90)
 			(hide yes)
@@
 			)
 		)
-		(property "Footprint" ""
+		(property "Footprint" "Resistor_SMD:R_1206_3216Metric"
 			(at 90.932 59.69 90)
 			(hide yes)
@@
 			)
 		)
-		(property "Footprint" ""
+		(property "Footprint" "Resistor_SMD:R_1206_3216Metric"
 			(at 238.252 59.69 90)
 			(hide yes)
@@
 			)
 		)
-		(property "Footprint" ""
+		(property "Footprint" "Resistor_SMD:R_1206_3216Metric"
 			(at 70.612 59.69 90)
 			(hide yes)
@@
 				(path "/c25060f1-f2f3-4cbd-b6ee-5f66e19502f5"
 					(reference "R3")
+					(unit 1)
+				)
+			)
+		)
+	)
+	(symbol
+		(lib_id "Connector:Screw_Terminal_01x04")
+		(at 140.97 76.2 90)
+		(unit 1)
+		(body_style 1)
+		(exclude_from_sim no)
+		(in_bom yes)
+		(on_board yes)
+		(in_pos_files yes)
+		(dnp no)
+		(fields_autoplaced yes)
+		(property "Reference" "J3"
+			(at 142.24 69.85 90)
+			(show_name no)
+			(do_not_autoplace no)
+			(effects
+				(font
+					(size 1.27 1.27)
+				)
+			)
+		)
+		(property "Value" "Screw_Terminal_01x04"
+			(at 142.24 72.39 90)
+			(show_name no)
+			(do_not_autoplace no)
+			(effects
+				(font
+					(size 1.27 1.27)
+				)
+			)
+		)
+		(property "Footprint" ""
+			(at 140.97 76.2 0)
+			(hide yes)
+			(show_name no)
+			(do_not_autoplace no)
+			(effects
+				(font
+					(size 1.27 1.27)
+				)
+			)
+		)
+		(property "Datasheet" ""
+			(at 140.97 76.2 0)
+			(hide yes)
+			(show_name no)
+			(do_not_autoplace no)
+			(effects
+				(font
+					(size 1.27 1.27)
+				)
+			)
+		)
+		(property "Description" "Generic screw terminal, single row, 01x04, script generated (kicad-library-utils/schlib/autogen/connector/)"
+			(at 140.97 76.2 0)
+			(hide yes)
+			(show_name no)
+			(do_not_autoplace no)
+			(effects
+				(font
+					(size 1.27 1.27)
+				)
+			)
+		)
+		(pin "1"
+		)
+		(pin "3"
+		)
+		(pin "4"
+		)
+		(pin "2"
+		)
+		(instances
+			(project "Stepper Motor Driver"
+				(path "/c25060f1-f2f3-4cbd-b6ee-5f66e19502f5"
+					(reference "J3")
 					(unit 1)
 				)
@@
 			)
 		)
-		(property "Footprint" ""
+		(property "Footprint" "Capacitor_SMD:C_1206_3216Metric"
 			(at 71.12 53.6448 0)
 			(hide yes)
@@
 			)
 		)
-		(property "Footprint" ""
+		(property "Footprint" "Capacitor_SMD:C_1206_3216Metric"
 			(at 30.48 53.6448 0)
 			(hide yes)
@@
 			)
 		)
-		(property "Footprint" ""
+		(property "Footprint" "Resistor_SMD:R_1206_3216Metric"
 			(at 198.882 59.69 90)
 			(hide yes)
@@
 			)
 		)
-		(property "Footprint" ""
+		(property "Footprint" "Capacitor_SMD:C_1206_3216Metric"
 			(at 218.44 53.6448 0)
 			(hide yes)
@@
 				)
 			)
+		)
+	)
+	(sheet
+		(at 194.31 120.65)
+		(size 35.56 12.7)
+		(exclude_from_sim no)
+		(in_bom yes)
+		(on_board yes)
+		(dnp no)
+		(fields_autoplaced yes)
+		(stroke
+			(width 0.1524)
+			(type solid)
+		)
+		(fill
+			(color 0 0 0 0)
+		)
+		(property "Sheetname" "Power"
+			(at 194.31 119.9384 0)
+			(show_name no)
+			(do_not_autoplace no)
+			(effects
+				(font
+					(size 1.27 1.27)
+				)
+				(justify left bottom)
+			)
+		)
+		(property "Sheetfile" "Power.kicad_sch"
+			(at 194.31 133.9346 0)
+			(show_name no)
+			(do_not_autoplace no)
+			(effects
+				(font
+					(size 1.27 1.27)
+				)
+				(justify left top)
+			)
+		)
+		(instances
+			(project "Stepper Motor Driver"
+				(path "/c25060f1-f2f3-4cbd-b6ee-5f66e19502f5"
+					(page "10")
+				)
+			)

Commit message: Better buck converters and rest of power architecture
Changed lines of the file:
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@@
 	(text "Connect terminal 1 to coil A and back to terminal 2.\nConnect terminal 3 to coil B and back to terminal 4.\n"
 		(exclude_from_sim no)
-		(at 141.986 86.868 0)
+		(at 141.732 86.868 0)
 		(effects
 			(font

Commit message: Fixed missing PWR_FLAG
Parts:
- removed J1, J2: Conn_01x22_Socket, Connector_PinSocket_2.54mm:PinSocket_1x22_P2.54mm_Vertical, symbol Connector:Conn_01x22_Socket
Other:
- sheet Power ports: added 24V, GND; removed none
Changed lines of the file:
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@@
-	)
-	(symbol
-		(lib_id "Connector:Conn_01x22_Socket")
-		(at 55.88 165.1 90)
-		(unit 1)
-		(body_style 1)
-		(exclude_from_sim no)
-		(in_bom yes)
-		(on_board yes)
-		(in_pos_files yes)
-		(dnp no)
-		(property "Reference" "J2"
-			(at 57.15 162.56 90)
-			(show_name no)
-			(do_not_autoplace no)
-			(effects
-				(font
-					(size 1.27 1.27)
-				)
-			)
-		)
-		(property "Value" "Conn_01x22_Socket"
-			(at 57.15 160.02 90)
-			(show_name no)
-			(do_not_autoplace no)
-			(effects
-				(font
-					(size 1.27 1.27)
-				)
-			)
-		)
-		(property "Footprint" "Connector_PinSocket_2.54mm:PinSocket_1x22_P2.54mm_Vertical"
-			(at 55.88 164.084 90)
-			(show_name no)
-			(do_not_autoplace no)
-			(effects
-				(font
-					(size 1.27 1.27)
-				)
-			)
-		)
-		(property "Datasheet" ""
-			(at 55.88 165.1 0)
-			(hide yes)
-			(show_name no)
-			(do_not_autoplace no)
-			(effects
-				(font
-					(size 1.27 1.27)
-				)
-			)
-		)
-		(property "Description" "Generic connector, single row, 01x22, script generated"
-			(at 55.88 165.1 0)
-			(hide yes)
-			(show_name no)
-			(do_not_autoplace no)
-			(effects
-				(font
-					(size 1.27 1.27)
-				)
-			)
-		)
-		(pin "16"
-		)
-		(pin "18"
-		)
-		(pin "1"
-		)
-		(pin "2"
-		)
-		(pin "10"
-		)
-		(pin "4"
-		)
-		(pin "11"
-		)
-		(pin "9"
-		)
-		(pin "3"
-		)
-		(pin "13"
-		)
-		(pin "15"
-		)
-		(pin "12"
-		)
-		(pin "6"
-		)
-		(pin "14"
-		)
-		(pin "7"
-		)
-		(pin "5"
-		)
-		(pin "8"
-		)
-		(pin "17"
-		)
-		(pin "20"
-		)
-		(pin "19"
-		)
-		(pin "22"
-		)
-		(pin "21"
-		)
-		(instances
-			(project "Stepper Motor Driver"
-				(path "/c25060f1-f2f3-4cbd-b6ee-5f66e19502f5"
-					(reference "J2")
-					(unit 1)
-				)
-			)
-		)
 	)
 	(symbol
@@
 				(path "/c25060f1-f2f3-4cbd-b6ee-5f66e19502f5"
 					(reference "R1")
-					(unit 1)
-				)
-			)
-		)
-	)
-	(symbol
-		(lib_id "Connector:Conn_01x22_Socket")
-		(at 58.42 144.78 270)
-		(unit 1)
-		(body_style 1)
-		(exclude_from_sim no)
-		(in_bom yes)
-		(on_board yes)
-		(in_pos_files yes)
-		(dnp no)
-		(property "Reference" "J1"
-			(at 57.15 147.32 90)
-			(show_name no)
-			(do_not_autoplace no)
-			(effects
-				(font
-					(size 1.27 1.27)
-				)
-			)
-		)
-		(property "Value" "Conn_01x22_Socket"
-			(at 57.15 149.86 90)
-			(show_name no)
-			(do_not_autoplace no)
-			(effects
-				(font
-					(size 1.27 1.27)
-				)
-			)
-		)
-		(property "Footprint" "Connector_PinSocket_2.54mm:PinSocket_1x22_P2.54mm_Vertical"
-			(at 58.42 145.796 90)
-			(show_name no)
-			(do_not_autoplace no)
-			(effects
-				(font
-					(size 1.27 1.27)
-				)
-			)
-		)
-		(property "Datasheet" ""
-			(at 58.42 144.78 0)
-			(hide yes)
-			(show_name no)
-			(do_not_autoplace no)
-			(effects
-				(font
-					(size 1.27 1.27)
-				)
-			)
-		)
-		(property "Description" "Generic connector, single row, 01x22, script generated"
-			(at 58.42 144.78 0)
-			(hide yes)
-			(show_name no)
-			(do_not_autoplace no)
-			(effects
-				(font
-					(size 1.27 1.27)
-				)
-			)
-		)
-		(pin "16"
-		)
-		(pin "18"
-		)
-		(pin "1"
-		)
-		(pin "2"
-		)
-		(pin "10"
-		)
-		(pin "4"
-		)
-		(pin "11"
-		)
-		(pin "9"
-		)
-		(pin "3"
-		)
-		(pin "13"
-		)
-		(pin "15"
-		)
-		(pin "12"
-		)
-		(pin "6"
-		)
-		(pin "14"
-		)
-		(pin "7"
-		)
-		(pin "5"
-		)
-		(pin "8"
-		)
-		(pin "17"
-		)
-		(pin "20"
-		)
-		(pin "19"
-		)
-		(pin "22"
-		)
-		(pin "21"
-		)
-		(instances
-			(project "Stepper Motor Driver"
-				(path "/c25060f1-f2f3-4cbd-b6ee-5f66e19502f5"
-					(reference "J1")
 					(unit 1)
 				)
@@
 	)
 	(sheet
-		(at 194.31 120.65)
+		(at 31.75 97.79)
 		(size 35.56 12.7)
 		(exclude_from_sim no)
@@
 		)
 		(property "Sheetname" "Power"
-			(at 194.31 119.9384 0)
+			(at 31.75 97.0784 0)
 			(show_name no)
 			(do_not_autoplace no)
@@
 		)
 		(property "Sheetfile" "Power.kicad_sch"
-			(at 194.31 133.9346 0)
+			(at 31.75 111.0746 0)
 			(show_name no)
 			(do_not_autoplace no)
@@
 			)
 		)
+		(pin "24V" input
+			(at 67.31 101.6 0)
+			(effects
+				(font
+					(size 1.27 1.27)
+				)
+				(justify right)
+			)
+		)
+		(pin "GND" input
+			(at 67.31 106.68 0)
+			(effects
+				(font
+					(size 1.27 1.27)
+				)
+				(justify right)
+			)
+		)

Commit message: Adding test points and FPGA sockets
Parts:
- added J1, J2: Conn_01x24_Socket, Connector_PinHeader_2.54mm:PinHeader_1x27_P2.54mm_Vertical, symbol Connector:Conn_01x24_Socket
