File: electrical/Stepper-Motor-Driver/circuits/H-Bridge Controller.kicad_sch (KiCad schematic)
At the start: 0 parts

Commit message: Current sensing circuit
Changed lines of the file:
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@@
 		)
 	)
-	(hierarchical_label "BRB"
-		(shape input)
+	(hierarchical_label "BR2"
+		(shape bidirectional)
 		(at 82.55 45.72 270)
 		(effects
@@
 		)
 	)
-	(hierarchical_label "HIB"
+	(hierarchical_label "HI2"
 		(shape input)
 		(at 129.54 26.67 0)
@@
 		)
 	)
-	(hierarchical_label "LIB"
+	(hierarchical_label "LI2"
 		(shape input)
 		(at 129.54 29.21 0)
@@
 		)
 	)
-	(hierarchical_label "BRA"
-		(shape input)
+	(hierarchical_label "BR1"
+		(shape bidirectional)
 		(at 71.12 45.72 270)
 		(effects
@@
 		)
 	)
-	(hierarchical_label "HIA"
+	(hierarchical_label "HI1"
 		(shape input)
 		(at 22.86 26.67 180)
@@
 		)
 	)
-	(hierarchical_label "LIA"
+	(hierarchical_label "LI1"
 		(shape input)
 		(at 22.86 29.21 180)
@@
 			)
 		)
-		(pin "OUT" input
+		(pin "OUT" bidirectional
 			(at 90.17 27.94 180)
 			(effects
@@
 			)
 		)
-		(pin "OUT" input
+		(pin "OUT" bidirectional
 			(at 62.23 27.94 0)
 			(effects

Commit message: Initial PCB layout
Parts:
- added C31: 470uF, Capacitor_THT:CP_Radial_D12.5mm_P5.00mm, symbol Device:C_Polarized
- added C33: 1uF, Capacitor_SMD:C_1206_3216Metric, symbol Device:C
- added C35: 100nF, Capacitor_SMD:C_1206_3216Metric, symbol Device:C
Connections:
- new net +VMotor: C31.1, C33.1, C35.1
- new net GND: C31.2, C33.2, C35.2
Other:
- sheet Left Half-Bridge Controller ports: added +VMotorIn; removed none
- sheet Right Half-Bridge Controller ports: added +VMotorIn; removed none
